File: Kicad.kicad_pcb (KiCad board)
At the start: 4 copper layers, 54 x 54.5 mm, 35 parts, among them J1 Conn_02x07_Odd_Even, J2 Conn_01x02, J3 Conn_01x04, J4 Conn_01x02, J42 Conn_01x04, J5 Conn_01x02, J52 Conn_01x04, J6 Conn_01x03, J62 Conn_01x03, U1 STM32L021K4Tx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

Commit message: Plus compact pas fini
Parts:
- moved AE2 48.6 mm to (142.1, 80.2)
- moved J52 37.1 mm to (155.5, 74.4), turned to -90 degrees
- moved U2 36.7 mm to (157.5, 114.0), turned to -90 degrees
- moved D1 34.8 mm to (160.5, 99.1), turned to 90 degrees
- moved J4 33.6 mm to (179.2, 80.3), turned to -90 degrees
- moved J2 32.1 mm to (159.2, 106.3), turned to -90 degrees
- moved J42 31.7 mm to (165.0, 111.7), turned to 180 degrees
- moved EM 28.9 mm to (157.0, 81.1)
- moved L1 27.0 mm to (166.5, 84.2)
- moved J1 26.8 mm to (145.1, 90.6), turned to -90 degrees
- moved C9 25.3 mm to (160.4, 114.0), turned to 90 degrees
- moved AE1 23.8 mm to (177.7, 71.8)
- moved C2 23.8 mm to (168.8, 86.7)
- moved C8 22.7 mm to (157.5, 109.8), turned to -90 degrees
- moved R2 22.0 mm to (170.2, 88.9), turned to 180 degrees
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- renumbered TP6 to EM, TP3 to PC, TP2 to REP
Routing:
- net NRST: track 0.00 -> 51.5 mm
- net TX Dati: track 0.00 -> 44.6 mm
- net GND: track 8.56 -> 50.7 mm
- net SYS_SWCLK: track 0.00 -> 31.0 mm
- net SYS_SWDIO: track 0.00 -> 28.0 mm
- net USART_RX: track 0.00 -> 25.1 mm
- net DATA_REC: track 0.00 -> 23.3 mm
- net +3.3V: track 0.00 -> 19.8 mm, vias 0 -> 1
- net Net-(AE2-A): track 0.00 -> 14.3 mm
- net PC: track 0.00 -> 12.3 mm
- net +5V: track 0.00 -> 9.74 mm
- net +3.3VA: track 0.00 -> 6.93 mm
- net Net-(AE1-A): track 2.56 -> 9.10 mm
- net USART_TX: track 0.00 -> 4.77 mm, vias 0 -> 2
- net SDA: track 0.00 -> 4.56 mm
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
Commit message: test
Parts:
- removed H4: MountingHole_Pad, MountingHole:MountingHole_3.2mm_M3_DIN965_Pad
- moved H3 53.3 mm to (172.0, 80.7)
- moved C9 9.63 mm to (160.4, 104.4), turned to 180 degrees
- moved U2 7.30 mm to (160.4, 107.3), turned to 0 degrees
- moved J2 6.53 mm to (152.7, 105.6), turned to 0 degrees
- moved H2 4.65 mm to (139.5, 76.6)
- moved H1 4.22 mm to (145.9, 105.7)
- moved J3 3.60 mm to (172.1, 95.8)
- moved AE2 3.52 mm to (145.2, 81.9)
- moved AE1 3.00 mm to (177.6, 74.8)
- moved C8 2.88 mm to (156.2, 107.3), turned to 0 degrees
- moved R7 2.74 mm to (167.5, 93.9)
- moved R3 2.72 mm to (155.3, 99.5)
- moved C1 2.67 mm to (155.3, 97.7)
- moved C4 2.67 mm to (155.3, 96.1)
- moved C5 2.67 mm to (159.4, 83.4)
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Routing:
- net GND: track 50.7 -> 202.2 mm, vias 0 -> 3
- net +3.3V: track 19.8 -> 124.4 mm
- net USART_TX: track 4.77 -> 28.1 mm
- net TX Dati: track 44.6 -> 62.3 mm
- net SCL: track 3.50 -> 9.57 mm
- net SDA: track 4.56 -> 10.6 mm
- net +5V: track 9.74 -> 13.2 mm
- net Net-(AE1-A): track 9.10 -> 5.84 mm
- net DATA_REC: track 23.3 -> 20.2 mm
- net Net-(AE2-A): track 14.3 -> 13.3 mm
- net NRST: track 51.5 -> 52.2 mm
Other:
- board size 54 x 54.5 mm -> 47 x 45.6 mm
