File: Kicad-emeteur/Kicad/Kicad.kicad_pcb (KiCad board)
At the start: 4 copper layers, 32 x 28.2 mm, 26 parts, among them J1 Conn_02x07_Odd_Even, J2 Conn_01x02, J5 Conn_01x02, J52 Conn_01x04, J6 Conn_01x03, J62 Conn_01x03, U1 STM32L021K4Tx, U2 BU33SD5WG-TR

Commit message: feat: Add initial KiCad project files for the emitter.
Routing:
- net GND: track 150.9 -> 80.3 mm
- net +3.3V: track 81.3 -> 52.3 mm
Changed lines of the file:
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@@
-	)
-	(segment
-		(start 113.529 97.911)
-		(end 113.529 114.719)
-		(width 0.2)
-		(layer "In2.Cu")
-		(net 2)
-	)
-	(segment
-		(start 115.84 95.6)
-		(end 113.529 97.911)
-		(width 0.2)
-		(layer "In2.Cu")
-		(net 2)
-	)
-	(segment
-		(start 111.01 115.87)
-		(end 108.47 113.33)
-		(width 0.2)
-		(layer "In2.Cu")
-		(net 2)
-	)
-	(segment
-		(start 113.529 114.719)
-		(end 114.68 115.87)
-		(width 0.2)
-		(layer "In2.Cu")
-		(net 2)
-	)
-	(segment
-		(start 114.68 115.87)
-		(end 111.01 115.87)
-		(width 0.2)
-		(layer "In2.Cu")
-		(net 2)
 	)
 	(segment
@@
 		(width 0.2)
 		(layer "F.Cu")
-		(net 3)
-	)
-	(segment
-		(start 114.68 118.41)
-		(end 111.01 118.41)
-		(width 0.2)
-		(layer "In1.Cu")
-		(net 3)
-	)
-	(segment
-		(start 111.01 118.41)
-		(end 105.93 113.33)
-		(width 0.2)
-		(layer "In1.Cu")
-		(net 3)
-	)
-	(segment
-		(start 105.93 113.33)
-		(end 102.9725 113.33)
-		(width 0.2)
-		(layer "In1.Cu")
-		(net 3)
-	)
-	(segment
-		(start 115.87 117.22)
-		(end 114.68 118.41)
-		(width 0.2)
-		(layer "In1.Cu")
-		(net 3)
-	)
-	(segment
-		(start 122.309 96.751)
-		(end 119.531 96.751)
-		(width 0.2)
-		(layer "In1.Cu")
-		(net 3)
-	)
-	(segment
-		(start 103.97 96.97)
-		(end 99.48 96.97)
-		(width 0.2)
-		(layer "In1.Cu")
-		(net 3)
-	)
-	(segment
-		(start 119.531 96.751)
-		(end 118.38 95.6)
-		(width 0.2)
-		(layer "In1.Cu")
-		(net 3)
-	)
-	(segment
-		(start 117.229 96.751)
-		(end 106.491 96.751)
-		(width 0.2)
-		(layer "In1.Cu")
-		(net 3)
-	)
-	(segment
-		(start 105.93 107.690108)
-		(end 99.48 101.240108)
-		(width 0.2)
-		(layer "In1.Cu")
-		(net 3)
-	)
-	(segment
-		(start 105.93 113.33)
-		(end 105.93 107.690108)
-		(width 0.2)
-		(layer "In1.Cu")
-		(net 3)
-	)
-	(segment
-		(start 123.52 117.22)
-		(end 115.87 117.22)
-		(width 0.2)
-		(layer "In1.Cu")
-		(net 3)
-	)
-	(segment
-		(start 105.34 95.6)
-		(end 103.97 96.97)
-		(width 0.2)
-		(layer "In1.Cu")
-		(net 3)
-	)
-	(segment
-		(start 102.9725 113.33)
-		(end 101.595 114.7075)
-		(width 0.2)
-		(layer "In1.Cu")
-		(net 3)
-	)
-	(segment
-		(start 123.46 95.6)
-		(end 122.309 96.751)
-		(width 0.2)
-		(layer "In1.Cu")
-		(net 3)
-	)
-	(segment
-		(start 106.491 96.751)
-		(end 105.34 95.6)
-		(width 0.2)
-		(layer "In1.Cu")
-		(net 3)
-	)
-	(segment
-		(start 99.48 101.240108)
-		(end 99.48 96.97)
-		(width 0.2)
-		(layer "In1.Cu")
-		(net 3)
-	)
-	(segment
-		(start 118.38 95.6)
-		(end 117.229 96.751)
-		(width 0.2)
-		(layer "In1.Cu")
 		(net 3)
 	)
@@
 	)
 	(segment
-		(start 108.579 112.179)
-		(end 113.529 112.179)
+		(start 112.81776 113.9)
+		(end 114.11 113.9)
 		(width 0.2)
 		(layer "B.Cu")
@@
 	)
 	(segment
-		(start 113.529 112.179)
-		(end 114.68 113.33)
+		(start 110.80776 111.89)
+		(end 112.81776 113.9)
 		(width 0.2)
 		(layer "B.Cu")
@@
 	)
 	(segment
+		(start 110 111.89)
+		(end 110.80776 111.89)
+		(width 0.2)
+		(layer "B.Cu")
+		(net 20)
+	)
+	(segment
 		(start 98.31 101.91)
-		(end 108.579 112.179)
+		(end 100.02 101.91)
 		(width 0.2)
 		(layer "B.Cu")
+		(net 20)
+	)
+	(segment
+		(start 114.11 113.9)
+		(end 114.68 113.33)
+		(width 0.2)
+		(layer "B.Cu")
+		(net 20)
+	)
+	(segment
+		(start 100.02 101.91)
+		(end 110 111.89)
+		(width 0.2)
+		(layer "B.Cu")
