File: Kicad-recepteur/Kicad/Kicad.kicad_sch (KiCad schematic)
At the start: 25 parts, among them J1 Conn_02x07_Odd_Even, J2 Conn_01x02, J3 Conn_01x04, J4 Conn_01x02, J42 Conn_01x04, U1 STM32L021K4Tx, U2 BU33SD5WG-TR

Commit message: feat: Add initial KiCad PCB and schematic files for the receiver project.
Parts:
- removed J2: Conn_01x02, Connector_PinSocket_2.54mm:PinSocket_1x02_P2.54mm_Vertical, symbol Connector_Generic:Conn_01x02
- added J5: USB_C_Receptacle_PowerOnly_6P, Connector_USB:USB_C_Receptacle_GCT_USB4125-xx-x-0190_6P_TopMnt_Horizontal, symbol Connector:USB_C_Receptacle_PowerOnly_6P
- added R1, R5: 5.1k, Resistor_SMD:R_0603_1608Metric_Pad0.98x0.95mm_HandSolder, symbol Device:R
Connections:
- net +5V: now also J5.A9 (VBUS), J5.B9 (VBUS)
- net GND: now also J5.A12 (GND), J5.B12 (GND), J5.S1 (SHIELD), R1.2, R5.2
- new net: J5.B5 (CC2), R1.1
- new net: J5.A5 (CC1), R5.1
Other:
- note removed: "Connecteur alim 5V"
- moved on the sheet: C1, C16, C2, C4, C5, C6, C8, C9, D1, L1, R2, R3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
